Commit message: Update load escher

File: escher_description/robot/escher.urdf (robot description, URDF)
Before this commit: robot escher, 49 links, 48 joints
Links:
- link chest: mass 15.967544717148 -> 9.867544717148; geometry collision box size=0.24 0.43 0.325; visual mesh filename=package://escher_description/robot/meshes/chest.stl scale=.001 .001 .001
- link head: geometry collision box size=0.155386 0.122 0.2991; visual mesh filename=package://escher_description/robot/meshes/head.stl scale=.001 .001 .001
- link head_lidar: geometry collision box size=0.1395 0.06 0.093; visual mesh filename=package://escher_description/robot/meshes/head_lidar.stl scale=.001 .001 .001
- link l_arm: geometry collision cylinder length=0.32 radius=0.05; visual mesh filename=package://escher_description/robot/meshes/ShoulderYawLeft.s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 scale=.001 .001 .001
- link l_elbow_link: geometry visual mesh filename=package://escher_description/robot/meshes/ElbowLeft.stl scale=.001 .001 .001
- link l_foot: geometry collision box size=0.25 0.1485 0.05493235; visual mesh filename=package://escher_description/robot/meshes/l_foot.stl scale=.001 .001 .001
- link l_forearm: geometry collision cylinder length=0.1 radius=0.05; visual mesh filename=package://escher_description/robot/meshes/WristYawLeft.stl scale=.001 .001 .001
- link l_foreforearm: geometry collision cylinder length=0.08 radius=0.05; visual mesh filename=package://escher_description/robot/meshes/WristPitchRollLef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 scale=.001 .001 .001
- link l_index_link: geometry collision cylinder length=0.1 radius=0.025; visual mesh filename=package://escher_description/robot/meshes/PointerLeft.stl scale=.001 .001 .001
- link l_palm: geometry collision box size=0.18 0.071 0.105; visual mesh filename=package://escher_description/robot/meshes/PalmLeft.stl scale=.001 .001 .001
- link l_ring_link: geometry collision cylinder length=0.1 radius=0.025; visual mesh filename=package://escher_description/robot/meshes/RingLeft.stl scale=.001 .001 .001
- link l_shin: geometry collision box size=0.13 0.16 0.4512008; visual mesh filename=package://escher_description/robot/meshes/l_shin.stl scale=.001 .001 .001
- link l_shoulder: geometry collision cylinder length=0.2 radius=0.05; visual mesh filename=package://escher_description/robot/meshes/ShoulderPitchLeft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 scale=.001 .001 .001
- link l_shoulder_roll_link: geometry visual mesh filename=package://escher_description/robot/meshes/ShoulderRollLeft.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 scale=.001 .001 .001
- link l_thigh: geometry collision box size=0.28 0.21 0.45; visual mesh filename=package://escher_description/robot/meshes/l_thigh.stl scale=.001 .001 .001
- link l_thumb_base: geometry visual mesh filename=package://escher_description/robot/meshes/ThumbBaseLeft.stl scale=.001 .001 .001
- link l_thumb_link: geometry collision cylinder length=0.1 radius=0.025; visual mesh filename=package://escher_description/robot/meshes/ThumbLeft.stl scale=.001 .001 .001
- link neck: geometry collision box size=0.0541 0.096 0.05405; visual mesh filename=package://escher_description/robot/meshes/neck.stl scale=.001 .001 .001
- link r_arm: geometry collision cylinder length=0.32 radius=0.05; visual mesh filename=package://escher_description/robot/meshes/ShoulderYawRight.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 scale=.001 .001 .001
- link r_elbow_link: geometry visual mesh filename=package://escher_description/robot/meshes/ElbowRight.stl scale=.001 .001 .001
- link r_foot: geometry collision box size=0.25 0.1485 0.05493235; visual mesh filename=package://escher_description/robot/meshes/r_foot.stl scale=.001 .001 .001
- link r_forearm: geometry collision cylinder length=0.1 radius=0.05; visual mesh filename=package://escher_description/robot/meshes/WristYawRight.stl scale=.001 .001 .001
- link r_foreforearm: geometry collision cylinder length=0.08 radius=0.05; visual mesh filename=package://escher_description/robot/meshes/WristPitchRollRig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 scale=.001 .001 .001
- link r_index_link: geometry collision cylinder length=0.1 radius=0.025; visual mesh filename=package://escher_description/robot/meshes/PointerRight.stl scale=.001 .001 .001
- link r_palm: geometry collision box size=0.18 0.071 0.105; visual mesh filename=package://escher_description/robot/meshes/PalmRight.stl scale=.001 .001 .001
- link r_ring_link: geometry collision cylinder length=0.1 radius=0.025; visual mesh filename=package://escher_description/robot/meshes/RingRight.stl scale=.001 .001 .001
- link r_shin: geometry collision box size=0.13 0.16 0.4512008; visual mesh filename=package://escher_description/robot/meshes/r_shin.stl scale=.001 .001 .001
- link r_shoulder: geometry collision cylinder length=0.2 radius=0.05; visual mesh filename=package://escher_description/robot/meshes/ShoulderPitchRigh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 scale=.001 .001 .001
- link r_shoulder_roll_link: geometry visual mesh filename=package://escher_description/robot/meshes/ShoulderRollRight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 scale=.001 .001 .001
- link r_thigh: geometry collision box size=0.28 0.21 0.45; visual mesh filename=package://escher_description/robot/meshes/r_thigh.stl scale=.001 .001 .001
- link r_thumb_base: geometry visual mesh filename=package://escher_description/robot/meshes/ThumbBaseRight.stl scale=.001 .001 .001
- link r_thumb_link: geometry collision cylinder length=0.1 radius=0.025; visual mesh filename=package://escher_description/robot/meshes/ThumbRight.stl scale=.001 .001 .001
- link torso: geometry collision box size=0.307 0.41 0.26; visual mesh filename=package://escher_description/robot/meshes/torso.stl scale=.001 .001 .001
Joints:
- joint l_wrist_yaw: limit lower=-1.57079632679 upper=1.57079632679 effort=60.0 velocity=2.0944 -> lower=-0.0002 upper=1.57079632679 effort=60.0 velocity=2.0944
- joint pitch_revolute_joint: limit lower=-0.0 effort=1000.0 velocity=1 -> lower=-0.5236 upper=0.5236 effort=1000.0 velocity=1
- joint r_wrist_yaw: limit lower=-1.57079632679 upper=1.57079632679 effort=60.0 velocity=2.0944 -> lower=-1.57079632679 upper=0.0002 effort=60.0 velocity=2.0944
- joint roll_revolute_joint: limit lower=-0.0 effort=1000.0 velocity=1 -> lower=-0.5236 upper=0.5236 effort=1000.0 velocity=1
